Commit message: Imported upstream version '1.12.0' of 'upstream'

File: pr2_description/robots/pr2.urdf.xacro (robot description, xacro)
@@ -24,5 +24,4 @@
   <!-- Head sensors -->
   <xacro:include filename="$(find pr2_description)/urdf/sensors/head_sensor_package.urdf.xacro" />
-  <xacro:include filename="$(find pr2_description)/urdf/sensors/kinect_prosilica_camera.urdf.xacro" />
   <!-- Camera sensors -->
   <xacro:include filename="$(find pr2_description)/urdf/sensors/wge100_camera.urdf.xacro" />
@@ -63,20 +62,4 @@
     <origin xyz="0 0.110 0.0546" rpy="0 0 0" />
   </xacro:projector_wg6802418_v0>
-  <!-- Base of Kinect/Prosilica Mount -->
-  <xacro:kinect_prosilica_camera_swept_back_v0 name="head_mount" parent="head_plate_frame" >
-    <origin xyz="-0.137376 0 0.091746" rpy="0 0 0" />
-    <!--
-          Was -0.1 0 0.09225, -0.138 0 0.09225 looks good front back and sheet metal on bolt pattern,
-          -0.138 0 0.06225 is where Prosilica FOV just clears the head.
-          This is 30 mm (!) below the position in SolidWorks.
-          Lowering the Prosilica by this amount in SW makes the FOV hit around the aluminum / plastic junction.
-          Turns out that head_plate_frame is in some random position in space.
-          It is [0.0232 0 0.0645 from its parent, head_tilt_link.
-          The distance from head_plate_frame to the head_kinect_prosilica is 137.376 mm X and 91.746 mm Z.
-          So the origin should in fact be -0.137376 0 0.091746.
-          John is changing the Prosilica FOV based on my numbers.
-          Just need to roscd and svn up.
-    -->
-  </xacro:kinect_prosilica_camera_swept_back_v0>
   <xacro:pr2_tilting_laser_v0 name="laser_tilt" parent="torso_lift_link" laser_calib_ref="0.0">
     <origin xyz="0.09893 0 0.227" rpy="0 0 0" />
@@ -139,3 +122,33 @@
     <origin xyz=".135 0 .044" rpy="${M_PI/2} ${-32.25*M_PI/180} 0" />
   </xacro:wge100_camera_v0>
+  <!-- Kinect models -->
+  <!-- Kinect2 xacro -->
+  <xacro:if value="$(optenv KINECT2 false)">
+    <xacro:include filename="$(find pr2_description)/urdf/sensors/kinect2.urdf.xacro" />
+    <xacro:kinect2_v0 name="head_mount" parent="head_plate_frame" >
+      <origin xyz="-0.137376 0 0.091746" rpy="0 0 0" />
+    </xacro:kinect2_v0>
+  </xacro:if>
+  <!-- Kinect1 xacro -->
+  <xacro:unless value="$(optenv KINECT2 false)">
+    <xacro:if value="$(optenv KINECT1 false)">
+      <xacro:include filename="$(find pr2_description)/urdf/sensors/kinect_prosilica_camera.urdf.xacro" />
+      <!-- Base of Kinect/Prosilica Mount -->
+      <xacro:kinect_prosilica_camera_swept_back_v0 name="head_mount" parent="head_plate_frame" >
+        <origin xyz="-0.137376 0 0.091746" rpy="0 0 0" />
+        <!--
+              Was -0.1 0 0.09225, -0.138 0 0.09225 looks good front back and sheet metal on bolt pattern,
+              -0.138 0 0.06225 is where Prosilica FOV just clears the head.
+              This is 30 mm (!) below the position in SolidWorks.
+              Lowering the Prosilica by this amount in SW makes the FOV hit around the aluminum / plastic junction.
+              Turns out that head_plate_frame is in some random position in space.
+              It is [0.0232 0 0.0645 from its parent, head_tilt_link.
+              The distance from head_plate_frame to the head_kinect_prosilica is 137.376 mm X and 91.746 mm Z.
+              So the origin should in fact be -0.137376 0 0.091746.
+              John is changing the Prosilica FOV based on my numbers.
+              Just need to roscd and svn up.
+        -->
+      </xacro:kinect_prosilica_camera_swept_back_v0>
+    </xacro:if>
+  </xacro:unless>
 </robot>
